File: eng/kicad/serenity-game-1/serenity-game-1.sch (KiCad schematic (older format))
At the start: 20 parts, among them J1 Conn_01x06_Male, SW1 SW_Push, SW2 SW_Push, SW3 SW_Push, SW4 SW_Push, SW5 SW_Push, U1 PIC16F690-IP

Commit message: Schematic addition of buttons and labeling of wires (WIP).
Parts:
- added J2: Conn_01x04_Female, symbol Connector:Conn_01x04_Female
- added SW10, SW8, SW9: SW_Push, Button_Switch_THT:SW_PUSH_6mm_H7.3mm, symbol Switch:SW_Push
- added SW6: SW_SPDT, Button_Switch_THT:SW_CuK_OS102011MA1QN1_SPDT_Angled, symbol Switch:SW_SPDT
- added SW7: SW_SP3T, symbol Switch:SW_SP3T
- BT1: footprint (none) -> Battery:BatteryHolder_Keystone_2479_3xAAA
- D1, D2, D3, D4: footprint (none) -> LED_THT:LED_D5.0mm
- J1: footprint (none) -> Connector_PinHeader_2.54mm:PinHeader_1x06_P2.54mm_Horizontal
- SW1, SW2, SW3, SW4, SW5: footprint (none) -> Button_Switch_THT:SW_PUSH_6mm_H7.3mm
Connections:
- net labels added: AUDIO, LED1_RED, LED2_YELLOW, LED3_GREEN, LED4_BLUE
- wire segments 0 -> 18
Changed lines of the file:
@@
 EESchema Schematic File Version 4
+LIBS:serenity-game-1-cache
 EELAYER 26 0
 EELAYER END
@@
 L MCU_Microchip_PIC16:PIC16F690-IP U1
 U 1 1 616C1FC2
-P 4400 3850
-F 0 "U1" H 4400 4828 50  0000 C CNN
-F 1 "PIC16F690-IP" H 4400 4737 50  0000 C CNN
-F 2 "Package_DIP:DIP-20_W7.62mm_Socket" H 4400 3850 50  0001 C CIN
-F 3 "http://ww1.microchip.com/downloads/en/DeviceDoc/41262E.pdf" H 4400 3850 50  0001 C CNN
-	1    4400 3850
+P 4400 3800
+F 0 "U1" H 4400 4778 50  0000 C CNN
+F 1 "PIC16F690-IP" H 4400 4687 50  0000 C CNN
+F 2 "Package_DIP:DIP-20_W7.62mm_Socket" H 4400 3800 50  0001 C CIN
+F 3 "http://ww1.microchip.com/downloads/en/DeviceDoc/41262E.pdf" H 4400 3800 50  0001 C CNN
+	1    4400 3800
 	1    0    0    -1
 $EndComp
@@
 L Device:C C1
 U 1 1 616C2198
-P 1800 3750
-F 0 "C1" H 1915 3796 50  0000 L CNN
-F 1 "C" H 1915 3705 50  0000 L CNN
-F 2 "Capacitor_THT:C_Disc_D3.0mm_W1.6mm_P2.50mm" H 1838 3600 50  0001 C CNN
-F 3 "~" H 1800 3750 50  0001 C CNN
-	1    1800 3750
+P 2100 2700
+F 0 "C1" H 2215 2746 50  0000 L CNN
+F 1 "C" H 2215 2655 50  0000 L CNN
+F 2 "Capacitor_THT:C_Disc_D3.0mm_W1.6mm_P2.50mm" H 2138 2550 50  0001 C CNN
+F 3 "~" H 2100 2700 50  0001 C CNN
+	1    2100 2700
 	1    0    0    -1
 $EndComp
@@
 L Device:Battery BT1
 U 1 1 616C2443
-P 1000 3750
-F 0 "BT1" H 1108 3796 50  0000 L CNN
-F 1 "Battery" H 1108 3705 50  0000 L CNN
-F 2 "" V 1000 3810 50  0001 C CNN
-F 3 "~" V 1000 3810 50  0001 C CNN
-	1    1000 3750
+P 900 2700
+F 0 "BT1" H 1008 2746 50  0000 L CNN
+F 1 "Battery" H 1008 2655 50  0000 L CNN
+F 2 "Battery:BatteryHolder_Keystone_2479_3xAAA" V 900 2760 50  0001 C CNN
+F 3 "~" V 900 2760 50  0001 C CNN
+	1    900  2700
 	1    0    0    -1
 $EndComp
@@
 F 0 "SW1" H 2450 6335 50  0000 C CNN
 F 1 "SW_Push" H 2450 6244 50  0000 C CNN
-F 2 "" H 2450 6250 50  0001 C CNN
+F 2 "Button_Switch_THT:SW_PUSH_6mm_H7.3mm" H 2450 6250 50  0001 C CNN
 F 3 "" H 2450 6250 50  0001 C CNN
 	1    2450 6050
@@
 F 0 "SW2" H 3350 6285 50  0000 C CNN
 F 1 "SW_Push" H 3350 6194 50  0000 C CNN
-F 2 "" H 3350 6200 50  0001 C CNN
+F 2 "Button_Switch_THT:SW_PUSH_6mm_H7.3mm" H 3350 6200 50  0001 C CNN
 F 3 "" H 3350 6200 50  0001 C CNN
 	1    3350 6000
@@
 F 0 "SW3" H 4200 6285 50  0000 C CNN
 F 1 "SW_Push" H 4200 6194 50  0000 C CNN
-F 2 "" H 4200 6200 50  0001 C CNN
+F 2 "Button_Switch_THT:SW_PUSH_6mm_H7.3mm" H 4200 6200 50  0001 C CNN
 F 3 "" H 4200 6200 50  0001 C CNN
 	1    4200 6000
@@
 F 0 "SW4" H 5200 6285 50  0000 C CNN
 F 1 "SW_Push" H 5200 6194 50  0000 C CNN
-F 2 "" H 5200 6200 50  0001 C CNN
+F 2 "Button_Switch_THT:SW_PUSH_6mm_H7.3mm" H 5200 6200 50  0001 C CNN
 F 3 "" H 5200 6200 50  0001 C CNN
 	1    5200 6000
@@
 F 0 "D1" H 7691 3366 50  0000 C CNN
 F 1 "LED" H 7691 3275 50  0000 C CNN
-F 2 "" H 7700 3150 50  0001 C CNN
+F 2 "LED_THT:LED_D5.0mm" H 7700 3150 50  0001 C CNN
 F 3 "~" H 7700 3150 50  0001 C CNN
 	1    7700 3150
@@
 F 0 "D4" H 7741 3966 50  0000 C CNN
 F 1 "LED" H 7741 3875 50  0000 C CNN
-F 2 "" H 7750 3750 50  0001 C CNN
+F 2 "LED_THT:LED_D5.0mm" H 7750 3750 50  0001 C CNN
 F 3 "~" H 7750 3750 50  0001 C CNN
 	1    7750 3750
@@
 F 0 "D2" H 7691 4566 50  0000 C CNN
 F 1 "LED" H 7691 4475 50  0000 C CNN
-F 2 "" H 7700 4350 50  0001 C CNN
+F 2 "LED_THT:LED_D5.0mm" H 7700 4350 50  0001 C CNN
 F 3 "~" H 7700 4350 50  0001 C CNN
 	1    7700 4350
@@
 F 0 "D3" H 7691 5116 50  0000 C CNN
 F 1 "LED" H 7691 5025 50  0000 C CNN
-F 2 "" H 7700 4900 50  0001 C CNN
+F 2 "LED_THT:LED_D5.0mm" H 7700 4900 50  0001 C CNN
 F 3 "~" H 7700 4900 50  0001 C CNN
 	1    7700 4900
@@
 L Connector:Conn_01x06_Male J1
 U 1 1 616C4412
-P 7500 1300
-F 0 "J1" H 7606 1678 50  0000 C CNN
-F 1 "Conn_01x06_Male" H 7606 1587 50  0000 C CNN
-F 2 "" H 7500 1300 50  0001 C CNN
-F 3 "~" H 7500 1300 50  0001 C CNN
-	1    7500 1300
+P 7500 1350
+F 0 "J1" H 7606 1728 50  0000 C CNN
+F 1 "Conn_01x06_Male" H 7606 1637 50  0000 C CNN
+F 2 "Connector_PinHeader_2.54mm:PinHeader_1x06_P2.54mm_Horizontal" H 7500 1350 50  0001 C CNN
+F 3 "~" H 7500 1350 50  0001 C CNN
+	1    7500 1350
 	1    0    0    -1
 $EndComp
@@
 F 0 "SW5" H 6650 2885 50  0000 C CNN
 F 1 "SW_Push" H 6650 2794 50  0000 C CNN
-F 2 "" H 6650 2800 50  0001 C CNN
+F 2 "Button_Switch_THT:SW_PUSH_6mm_H7.3mm" H 6650 2800 50  0001 C CNN
 F 3 "" H 6650 2800 50  0001 C CNN
 	1    6650 2600
@@
 Text Notes 3950 4000 0    50   ~ 0
 serenity game 1
+Wire Wire Line
+	2400 3400 2900 3400
+Wire Wire Line
+	2400 3300 2900 3300
+Wire Wire Line
+	2400 3500 2900 3500
+Wire Wire Line
+	2400 3600 2900 3600
+Wire Wire Line
+	2400 3800 2900 3800
+Wire Wire Line
+	2400 3700 2900 3700
+Wire Wire Line
+	2400 3900 2900 3900
+Wire Wire Line
+	2400 4000 2900 4000
+Wire Wire Line
+	5900 3400 6400 3400
+Wire Wire Line
+	5900 3300 6400 3300
+Wire Wire Line
+	5900 3500 6400 3500
+Wire Wire Line
+	5900 3600 6400 3600
+Wire Wire Line
+	5900 3800 6400 3800
+Wire Wire Line
+	5900 3700 6400 3700
+Wire Wire Line
+	5900 4100 6400 4100
+Wire Wire Line
+	5900 4000 6400 4000
+Wire Wire Line
+	5900 4300 6400 4300
+Wire Wire Line
+	5900 4200 6400 4200
+Text Label 2400 3700 0    50   ~ 0
+LED1_RED
+Text Label 2400 3800 0    50   ~ 0
+LED2_YELLOW
+Text Label 2400 3900 0    50   ~ 0
+LED3_GREEN
+Text Label 7850 4900 0    50   ~ 0
+LED3_GREEN
+Text Label -266950 192450 0    50   ~ 0
+LED4_BLUE
+Text Label 2400 4000 0    50   ~ 0
+LED4_BLUE
+Text Label 2400 3600 0    50   ~ 0
+AUDIO
+$Comp
+L Switch:SW_SPDT SW6
+U 1 1 61C3A92F
+P 1350 2200
+F 0 "SW6" H 1350 2485 50  0000 C CNN
+F 1 "SW_SPDT" H 1350 2394 50  0000 C CNN
+F 2 "Button_Switch_THT:SW_CuK_OS102011MA1QN1_SPDT_Angled" H 1350 2200 50  0001 C CNN
+F 3 "" H 1350 2200 50  0001 C CNN
+	1    1350 2200
+	1    0    0    -1
+$EndComp
+$Comp
+L Switch:SW_SP3T SW7
+U 1 1 61C3AB53
+P 2800 1850
+F 0 "SW7" H 2800 2133 50  0000 C CNN
+F 1 "SW_SP3T" H 2800 2042 50  0000 C CNN
+F 2 "" H 2175 2025 50  0001 C CNN
+F 3 "" H 2175 2025 50  0001 C CNN
+	1    2800 1850
+	1    0    0    -1
+$EndComp
+$Comp
+L Connector:Conn_01x04_Female J2
+U 1 1 61C3B835
+P 4100 1800
+F 0 "J2" H 4127 1776 50  0000 L CNN
+F 1 "Conn_01x04_Female" H 4127 1685 50  0000 L CNN
+F 2 "" H 4100 1800 50  0001 C CNN
+F 3 "~" H 4100 1800 50  0001 C CNN
+	1    4100 1800
+	1    0    0    -1
+$EndComp
+$Comp
+L Switch:SW_Push SW8
+U 1 1 61C3BD2D
+P 3300 1250
+F 0 "SW8" H 3300 1535 50  0000 C CNN
+F 1 "SW_Push" H 3300 1444 50  0000 C CNN
+F 2 "Button_Switch_THT:SW_PUSH_6mm_H7.3mm" H 3300 1450 50  0001 C CNN
+F 3 "" H 3300 1450 50  0001 C CNN
+	1    3300 1250
+	1    0    0    -1
+$EndComp
+$Comp
+L Switch:SW_Push SW9
+U 1 1 61C3BD33
+P 4200 1200
+F 0 "SW9" H 4200 1485 50  0000 C CNN
+F 1 "SW_Push" H 4200 1394 50  0000 C CNN
+F 2 "Button_Switch_THT:SW_PUSH_6mm_H7.3mm" H 4200 1400 50  0001 C CNN
+F 3 "" H 4200 1400 50  0001 C CNN
+	1    4200 1200
+	1    0    0    -1
+$EndComp
+$Comp
+L Switch:SW_Push SW10
+U 1 1 61C3BD39
+P 5050 1200
+F 0 "SW10" H 5050 1485 50  0000 C CNN
+F 1 "SW_Push" H 5050 1394 50  0000 C CNN
+F 2 "Button_Switch_THT:SW_PUSH_6mm_H7.3mm" H 5050 1400 50  0001 C CNN
+F 3 "" H 5050 1400 50  0001 C CNN
+	1    5050 1200
+	1    0    0    -1
+$EndComp
 $EndSCHEMATC
